File: MultiVib/i_trubni_multivib.sch (KiCad schematic (older format))
At the start: 10 parts

Commit message: labojums multi_vib
Parts:
- removed U?: DMC50601, symbol DMC50601
- added U1: EMX26, symbol EMX26
- gave numbers to parts that had none: 9
Connections:
- wire segments 31 -> 39
Changed lines of the file:
@@
 LIBS:device
 LIBS:transistors
+LIBS:dmc50601
 LIBS:conn
 LIBS:linear
@@
 LIBS:contrib
 LIBS:valves
-LIBS:jaunas
-LIBS:dmc50601
 LIBS:i_trubni_multivib-cache
 EELAYER 25 0
@@
 $EndDescr
 $Comp
-L CP1 C?
+L CP1 C2
 U 1 1 58C12733
 P 6400 4150
-F 0 "C?" H 6425 4250 50  0000 L CNN
+F 0 "C2" H 6425 4250 50  0000 L CNN
 F 1 "CP1" H 6425 4050 50  0000 L CNN
 F 2 "" H 6400 4150 50  0000 C CNN
@@
 $EndComp
 $Comp
-L CP1 C?
+L CP1 C1
 U 1 1 58C127A4
 P 5400 4150
-F 0 "C?" H 5425 4250 50  0000 L CNN
+F 0 "C1" H 5425 4250 50  0000 L CNN
 F 1 "CP1" H 5425 4050 50  0000 L CNN
 F 2 "" H 5400 4150 50  0000 C CNN
@@
 $EndComp
 $Comp
-L LED D?
+L LED D1
 U 1 1 58C12801
 P 5050 2950
-F 0 "D?" H 5050 3050 50  0000 C CNN
+F 0 "D1" H 5050 3050 50  0000 C CNN
 F 1 "LED" H 5050 2850 50  0000 C CNN
 F 2 "" H 5050 2950 50  0000 C CNN
@@
 $EndComp
 $Comp
-L LED D?
+L LED D2
 U 1 1 58C12870
 P 6850 3000
-F 0 "D?" H 6850 3100 50  0000 C CNN
+F 0 "D2" H 6850 3100 50  0000 C CNN
 F 1 "LED" H 6850 2900 50  0000 C CNN
 F 2 "" H 6850 3000 50  0000 C CNN
@@
 $EndComp
 $Comp
-L R R?
+L R R3
 U 1 1 58C128FD
 P 6050 3500
-F 0 "R?" V 6130 3500 50  0000 C CNN
+F 0 "R3" V 6130 3500 50  0000 C CNN
 F 1 "R" V 6050 3500 50  0000 C CNN
 F 2 "" V 5980 3500 50  0000 C CNN
@@
 $EndComp
 $Comp
-L R R?
+L R R2
 U 1 1 58C12AAC
 P 5650 3550
-F 0 "R?" V 5730 3550 50  0000 C CNN
+F 0 "R2" V 5730 3550 50  0000 C CNN
 F 1 "R" V 5650 3550 50  0000 C CNN
 F 2 "" V 5580 3550 50  0000 C CNN
@@
 $EndComp
 $Comp
-L R R?
+L R R4
 U 1 1 58C12B0F
 P 6850 3500
-F 0 "R?" V 6930 3500 50  0000 C CNN
+F 0 "R4" V 6930 3500 50  0000 C CNN
 F 1 "R" V 6850 3500 50  0000 C CNN
 F 2 "" V 6780 3500 50  0000 C CNN
@@
 $EndComp
 $Comp
-L R R?
+L R R1
 U 1 1 58C12B62
 P 5050 3450
-F 0 "R?" V 5130 3450 50  0000 C CNN
+F 0 "R1" V 5130 3450 50  0000 C CNN
 F 1 "R" V 5050 3450 50  0000 C CNN
 F 2 "" V 4980 3450 50  0000 C CNN
@@
 $EndComp
 $Comp
-L Battery BT?
+L Battery BT1
 U 1 1 58C133E6
 P 3900 4000
-F 0 "BT?" H 4000 4100 50  0000 L CNN
+F 0 "BT1" H 4000 4100 50  0000 L CNN
 F 1 "Battery" H 4000 4000 50  0000 L CNN
 F 2 "" V 3900 4060 50  0000 C CNN
@@
 	1    0    0    -1
 $EndComp
+$Comp
+L EMX26 U1
+U 1 1 58DD4C2F
+P 5875 4905
+F 0 "U1" H 6375 5225 60  0001 C CNN
+F 1 "EMX26" H 6455 5475 60  0000 C CNN
+F 2 "" H 5725 5355 60  0001 C CNN
+F 3 "http://www.mouser.com/ds/2/348/emx26-1017617.pdf" H 5725 5355 60  0001 C CNN
+	1    5875 4905
+	1    0    0    -1
+$EndComp
 Wire Wire Line
 	6850 2700 6850 2850
@@
 Wire Wire Line
 	5050 3600 5050 4650
-Wire Wire Line
-	5050 4650 6000 4650
 Connection ~ 5050 4150
 Wire Wire Line
-	6050 3650 6050 4750
+	5550 4150 5655 4150
+Wire Wire Line
+	6850 3350 6850 3150
+Wire Wire Line
+	6550 4150 6850 4150
+Wire Wire Line
+	6850 4655 6850 3650
+Connection ~ 6850 4150
+Wire Wire Line
+	3900 4200 3900 5405
+Wire Wire Line
+	6250 4150 6050 4150
+Wire Wire Line
+	6220 4645 5085 4645
+Wire Wire Line
+	5085 4645 5085 4650
+Wire Wire Line
+	5085 4650 5050 4650
+Wire Wire Line
+	6050 4505 5685 4505
+Wire Wire Line
+	6050 3650 6050 4505
+Wire Wire Line
+	5715 4915 5685 4915
+Wire Wire Line
+	5685 4915 5685 4505
+Wire Wire Line
+	6035 4915 6110 4915
+Wire Wire Line
+	6110 4915 6110 4570
+Wire Wire Line
+	6110 4570 5655 4570
+Wire Wire Line
+	5655 4570 5655 3700
+Wire Wire Line
+	5715 4975 5685 4975
+Wire Wire Line
+	5685 4975 5685 5050
+Wire Wire Line
+	5685 5050 6560 5050
+Wire Wire Line
+	3900 5405 6080 5405
+Wire Wire Line
+	6560 4655 6850 4655
+Wire Wire Line
+	6560 5050 6560 4655
+Wire Wire Line
+	5655 3700 5650 3700
+Connection ~ 5655 4150
 Connection ~ 6050 4150
 Wire Wire Line
-	5550 4150 5650 4150
-Connection ~ 5650 4150
-Wire Wire Line
-	6850 3350 6850 3150
-Wire Wire Line
-	6550 4150 6850 4150
-Wire Wire Line
-	6850 3650 6850 4650
-Wire Wire Line
-	6850 4650 6400 4650
-Connection ~ 6850 4150
-Wire Wire Line
-	6400 5400 6400 5050
-Wire Wire Line
-	3900 5400 6400 5400
-Wire Wire Line
-	5350 4700 5350 5400
-Wire Wire Line
-	3900 5400 3900 4200
-Connection ~ 5350 5400
-$Comp
-L DMC50601 U?
-U 1 1 58C9D1AD
-P 5300 5500
-F 0 "U?" H 5150 5950 60  0000 C CNN
-F 1 "DMC50601" H 5150 5950 60  0000 C CNN
-F 2 "" H 5150 5950 60  0001 C CNN
-F 3 "" H 5150 5950 60  0001 C CNN
-	1    5300 5500
-	1    0    0    -1
-$EndComp
-Wire Wire Line
-	5750 4700 5350 4700
-Wire Wire Line
-	6000 4650 6000 4700
-Wire Wire Line
-	6050 4750 6000 4750
-Wire Wire Line
-	6250 4150 6050 4150
-Wire Wire Line
-	5750 4800 5650 4800
-Wire Wire Line
-	5650 4800 5650 4150
-Wire Wire Line
-	6000 4800 6400 4800
-Wire Wire Line
-	6400 4800 6400 4650
-Wire Wire Line
-	5750 4750 5600 4750
-Wire Wire Line
-	5600 4750 5600 5050
-Wire Wire Line
-	5600 5050 6400 5050
+	5715 4865 5350 4865
+Wire Wire Line
+	5350 4865 5350 5405
+Connection ~ 5350 5405
+Wire Wire Line
+	6080 5405 6080 4975
+Wire Wire Line
+	6220 4645 6220 4855
+Wire Wire Line
+	6220 4855 6035 4855
+Wire Wire Line
+	6080 4975 6035 4975
 $EndSCHEMATC
