File: PWR_suplay/12v.sch (KiCad schematic (older format))
At the start: 3 parts, among them U1 LM7812ACT

Commit message: izlaboju teiktas kluas, tagad vajadzetu but
Changed lines of the file:
@@
 $EndDescr
-$Comp
-L GND #PWR01
-U 1 1 590F1D7E
-P 5170 3460
-F 0 "#PWR01" H 5170 3210 50  0001 C CNN
-F 1 "GND" H 5170 3310 50  0000 C CNN
-F 2 "" H 5170 3460 50  0000 C CNN
-F 3 "" H 5170 3460 50  0000 C CNN
-	1    5170 3460
-	1    0    0    -1
-$EndComp
 $Comp
 L CP1_Small C3
@@
 	5170 3345 5140 3345
 Wire Wire Line
-	5140 3345 5140 3390
+	5140 3345 5140 3460
 Connection ~ 5140 3390
-Wire Wire Line
-	5170 3460 5170 3390
-Connection ~ 5170 3390
 Wire Wire Line
 	5170 3280 5170 3345
@@
 	1    0    0    -1
 $EndComp
+$Comp
+L GND #PWR01
+U 1 1 590F1D7E
+P 5140 3460
+F 0 "#PWR01" H 5140 3210 50  0001 C CNN
+F 1 "GND" H 5140 3310 50  0000 C CNN
+F 2 "" H 5140 3460 50  0000 C CNN
+F 3 "" H 5140 3460 50  0000 C CNN
+	1    5140 3460
+	1    0    0    -1
+$EndComp
