File: PWR_suplay/220v.sch (KiCad schematic (older format))
At the start: 4 parts, among them P1 CONN_01X02, T1 Transformer_1P_1S

Commit message: izlaboju teiktas kluas, tagad vajadzetu but
Connections:
- net VCC renamed +220v
Changed lines of the file:
@@
 P 5560 1990
 F 0 "T1" H 5560 2240 50  0000 C CNN
-F 1 "Transformer_1P_1S" H 5560 1690 50  0000 C CNN
+F 1 "Transformer_1P_1S" H 5560 1690 50  0001 C CNN
 F 2 "" H 5560 1990 50  0000 C CNN
 F 3 "" H 5560 1990 50  0000 C CNN
@@
 P 4280 1980
 F 0 "P1" H 4280 2130 50  0000 C CNN
-F 1 "CONN_01X02" V 4380 1980 50  0000 C CNN
+F 1 "CONN_01X02" V 4380 1980 50  0001 C CNN
 F 2 "" H 4280 1980 50  0000 C CNN
 F 3 "" H 4280 1980 50  0000 C CNN
@@
 Connection ~ 7880 2470
 Text HLabel 8920 1895 2    60   Output ~ 0
-VCC
++220v
 Wire Wire Line
 	8920 1895 8640 1895
