File: PWR_suplay/9V.sch (KiCad schematic (older format))
At the start: 3 parts, among them U4 LM7809ACT

Commit message: izlaboju teiktas kluas, tagad vajadzetu but
Changed lines of the file:
@@
 Connection ~ 4535 3255
 Wire Wire Line
-	3455 3700 3455 3045
+	3455 2835 3455 3700
+Connection ~ 3455 3260
 Wire Wire Line
-	3455 3045 3465 3045
-Wire Wire Line
-	3465 3045 3465 2835
-Wire Wire Line
-	3465 2835 3460 2835
+	3460 2835 3455 2835
 $EndSCHEMATC
