File: single_transisto_AMP/single_transisto_AMP.kicad_pcb (KiCad board)
At the start: 2 copper layers, 57.2 x 29.2 mm, 11 parts, among them P1 CONN_01X01, P2 CONN_01X01, P3 CONN_01X01, P4 CONN_01X01, Q1 BC547

Commit message: celini un urbumi
Routing:
- net Net-(BT1-Pad2): track 0.00 -> 52.4 mm
- net Net-(C2-Pad1): track 0.00 -> 33.3 mm
- net Net-(C1-Pad2): track 0.00 -> 27.4 mm
- net Net-(BT1-Pad1): track 0.00 -> 17.6 mm
- net Net-(Q1-Pad3): track 0.00 -> 10.9 mm
- net Net-(C1-Pad1): track 0.00 -> 4.44 mm
- added copper zone on B.Cu, net Net-(BT1-Pad2)
Changed lines of the file:
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@@
   (general
     (links 13)
-    (no_connects 13)
-    (area 190.424999 97.714999 247.725001 127.075001)
+    (no_connects 1)
+    (area 190.424999 97.554999 247.725001 128.025)
     (thickness 1.6)
     (drawings 10)
-    (tracks 0)
+    (tracks 28)
     (zones 0)
     (modules 11)
@@
     (visible_elements 7FFEEFFF)
     (pcbplotparams
-      (layerselection 0x00030_80000001)
+      (layerselection 0x01020_80000001)
       (usegerberextensions false)
       (excludeedgelayer true)
@@
       (psa4output false)
       (plotreference true)
-      (plotvalue true)
+      (plotvalue false)
       (plotinvisibletext false)
       (padsonsilk false)
@@
       (outputformat 1)
       (mirror false)
-      (drillshape 1)
+      (drillshape 0)
       (scaleselection 1)
       (outputdirectory ""))
@@
     (uvia_dia 0.3)
     (uvia_drill 0.2)
-    (add_net "Net-(BT1-Pad1)")
-    (add_net "Net-(BT1-Pad2)")
     (add_net "Net-(C1-Pad1)")
     (add_net "Net-(C1-Pad2)")
@@
     (uvia_dia 0.3)
     (uvia_drill 0.2)
+    (add_net "Net-(BT1-Pad1)")
+    (add_net "Net-(BT1-Pad2)")
   )
   (module Capacitors_THT:CP_Axial_L10.0mm_D4.5mm_P15.00mm_Horizontal (layer F.Cu)
@@
     (descr "module 1 pin (ou trou mecanique de percage)")
     (tags DEV)
-    (fp_text reference P1 (at 3.81 0) (layer F.SilkS)
+    (fp_text reference P1 (at -3.29692 -0.11684) (layer F.SilkS)
       (effects (font (size 1 1) (thickness 0.15)))
     )
@@
     (descr "module 1 pin (ou trou mecanique de percage)")
     (tags DEV)
-    (fp_text reference P2 (at 3.81 0) (layer F.SilkS)
+    (fp_text reference P2 (at -3.50012 -0.01778) (layer F.SilkS)
       (effects (font (size 1 1) (thickness 0.15)))
     )
@@
     (descr "module 1 pin (ou trou mecanique de percage)")
     (tags DEV)
-    (fp_text reference P3 (at 0 -3.048) (layer F.SilkS)
+    (fp_text reference P3 (at 3.69824 0.46482) (layer F.SilkS)
       (effects (font (size 1 1) (thickness 0.15)))
     )
@@
     (descr "module 1 pin (ou trou mecanique de percage)")
     (tags DEV)
-    (fp_text reference P4 (at 0 -3.048) (layer F.SilkS)
+    (fp_text reference P4 (at 3.94462 0.44196) (layer F.SilkS)
       (effects (font (size 1 1) (thickness 0.15)))
     )
@@
   (module bibloteeka_footprint:Nr2_battery_holder_1775485 (layer F.Cu)
     (at 234.7938 121.59 180)
-    (fp_text reference BT1 (at -1.35 -5.41 180) (layer F.SilkS)
+    (fp_text reference BT1 (at -1.2738 -4.6988 180) (layer F.SilkS)
       (effects (font (size 1 1) (thickness 0.15)))
     )
@@
   (gr_line (start 247.65 123.19) (end 247.65 101.6) (layer Edge.Cuts) (width 0.15))
   (gr_line (start 194.31 127) (end 243.84 127) (layer Edge.Cuts) (width 0.15))
+  (segment (start 199.771 115.2652) (end 195.4022 115.2652) (width 0.1) (layer F.Cu) (net 1))
+  (segment (start 195.4022 115.2652) (end 195.3514 115.2144) (width 0.1) (layer F.Cu) (net 1))
+  (segment (start 221.4814 108.5596) (end 212.561398 108.5596) (width 0.1) (layer F.Cu) (net 2))
+  (segment (start 212.561398 108.5596) (end 209.995998 105.9942) (width 0.1) (layer F.Cu) (net 2))
+  (segment (start 209.995998 105.9942) (end 206.248 105.9942) (width 0.1) (layer F.Cu) (net 2))
+  (segment (start 206.248 105.9942) (end 204.47 104.2162) (width 0.1) (layer F.Cu) (net 2))
+  (segment (start 204.47 100.33) (end 204.47 101.744213) (width 0.1) (layer F.Cu) (net 2))
+  (segment (start 204.47 101.744213) (end 204.47 104.2162) (width 0.1) (layer F.Cu) (net 2))
+  (segment (start 204.47 100.33) (end 199.8358 100.33) (width 0.1) (layer F.Cu) (net 2))
+  (segment (start 199.8358 100.33) (end 199.771 100.2652) (width 0.1) (layer F.Cu) (net 2))
+  (segment (start 211.2772 104.2162) (end 213.6206 106.5596) (width 0.1) (layer F.Cu) (net 3))
+  (segment (start 213.6206 106.5596) (end 219.4814 106.5596) (width 0.1) (layer F.Cu) (net 3))
+  (segment (start 209.55 104.2162) (end 211.2772 104.2162) (width 0.1) (layer F.Cu) (net 3))
+  (segment (start 219.47 100.33) (end 229.7938 100.33) (width 0.1) (layer F.Cu) (net 3))
+  (segment (start 241.8588 100.33) (end 238.985119 100.33) (width 0.1) (layer F.Cu) (net 3))
+  (segment (start 238.985119 100.33) (end 229.7938 100.33) (width 0.1) (layer F.Cu) (net 3))
+  (segment (start 229.7938 123.19) (end 229.7938 122.12934) (width 0.1) (layer F.Cu) (net 4))
+  (segment (start 229.7938 122.12934) (end 229.7938 115.33) (width 0.1) (layer F.Cu) (net 4))
+  (segment (start 229.7938 115.33) (end 228.379587 115.33) (width 0.1) (layer F.Cu) (net 4))
+  (segment (start 228.379587 115.33) (end 227.273387 114.2238) (width 0.1) (layer F.Cu) (net 4))
+  (segment (start 227.273387 114.2238) (end 204.5462 114.2238) (width 0.1) (layer F.Cu) (net 4))
+  (segment (start 195.58 123.19) (end 204.5462 114.2238) (width 0.1) (layer F.Cu) (net 4))
+  (segment (start 204.5462 114.2238) (end 204.5462 108.1024) (width 0.1) (layer F.Cu) (net 4))
+  (segment (start 234.7938 121.59) (end 241.935 114.4488) (width 0.1) (layer F.Cu) (net 5))
+  (segment (start 241.935 114.4488) (end 241.935 106.9086) (width 0.1) (layer F.Cu) (net 5))
+  (segment (start 210.8708 108.1024) (end 213.328 110.5596) (width 0.1) (layer F.Cu) (net 6))
+  (segment (start 213.328 110.5596) (end 219.4814 110.5596) (width 0.1) (layer F.Cu) (net 6))
+  (segment (start 209.6262 108.1024) (end 210.8708 108.1024) (width 0.1) (layer F.Cu) (net 6))
+  (zone (net 4) (net_name "Net-(BT1-Pad2)") (layer B.Cu) (hatch edge 0.508)
+    (connect_pads (clearance 0.508))
+    (min_thickness 0.254)
+    (fill yes (arc_segments 16) (thermal_gap 0.508) (thermal_bridge_width 0.508))
+    (polygon
+      (pts
+        (xy 228.04374 126.9873) (xy 193.95694 127.00762) (xy 192.53962 126.58852) (xy 191.62268 125.88748) (xy 191.643 125.8824)
+        (xy 191.1731 125.30328) (xy 190.754 124.42952) (xy 190.55588 123.71578) (xy 190.48222 123.07824) (xy 190.50508 101.30536)
+        (xy 190.74638 100.18522) (xy 191.47282 98.96856) (xy 192.70472 98.13544) (xy 193.68516 97.85096) (xy 194.47256 97.79)
+        (xy 243.85016 97.79508) (xy 244.65026 97.8662) (xy 245.18112 98.02622) (xy 246.33682 98.7044) (xy 247.03532 99.50958)
+        (xy 247.5484 100.61194) (xy 247.65254 101.56952) (xy 247.62714 123.444) (xy 247.4722 124.29744) (xy 247.07342 125.17374)
+        (xy 246.5451 125.87224) (xy 245.61292 126.5809) (xy 244.75186 126.89586) (xy 243.64696 127.0127)
+      )
+    )
+  )
 )

Commit message: bom un svg faili pievienoti
Parts:
- Q1: footprint Transistors_OldSowjetAera:OldSowjetaera_Transistor_Type-II_BigPads -> Transistors_OldSowjetAera:OldSowjetaera_Transistor_Type-II_SmallPads
Routing:
- net Net-(C2-Pad1): track 33.3 -> 39.5 mm
Changed lines of the file:
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@@
   (general
     (links 13)
-    (no_connects 1)
+    (no_connects 0)
     (area 190.424999 97.554999 247.725001 128.025)
     (thickness 1.6)
     (drawings 10)
-    (tracks 28)
+    (tracks 30)
     (zones 0)
     (modules 11)
@@
     (mod_text_size 1 1)
     (mod_text_width 0.15)
-    (pad_size 1.4 1.4)
-    (pad_drill 0.7)
+    (pad_size 1.6 1.6)
+    (pad_drill 0.8)
     (pad_to_mask_clearance 0.2)
     (aux_axis_origin 0 0)
@@
       (net 5 "Net-(BT1-Pad1)"))
   )
-  (module Transistors_OldSowjetAera:OldSowjetaera_Transistor_Type-II_BigPads (layer F.Cu)
-    (at 219.4814 108.5596 270)
-    (fp_text reference Q1 (at 0.1 -8.1 540) (layer F.SilkS)
-      (effects (font (size 1 1) (thickness 0.15)))
-    )
-    (fp_text value BC547 (at 0.1 7.6 270) (layer F.Fab)
-      (effects (font (size 1 1) (thickness 0.15)))
-    )
-    (fp_circle (center -4.8 0) (end -4.8 0.4) (layer F.SilkS) (width 0.15))
-    (fp_circle (center 0 0) (end 4 0) (layer F.SilkS) (width 0.15))
-    (fp_circle (center 0 0) (end 5.6 0) (layer F.SilkS) (width 0.15))
-    (pad 2 thru_hole oval (at 0 -2 270) (size 1.4 2.5) (drill 0.8) (layers *.Cu *.Mask)
-      (net 2 "Net-(C1-Pad2)"))
-    (pad 1 thru_hole oval (at -2 0) (size 1.4 2.5) (drill 0.8) (layers *.Cu *.Mask)
-      (net 3 "Net-(C2-Pad1)"))
-    (pad 3 thru_hole oval (at 2 0) (size 1.4 2.5) (drill 0.8) (layers *.Cu *.Mask)
-      (net 6 "Net-(Q1-Pad3)"))
-    (model Transistors_OldSowjetAera.3dshapes/OldSowjetaera_Transistor_Type-II_BigPads.wrl
-      (at (xyz 0 0 0))
-      (scale (xyz 0.3937 0.3937 0.3937))
-      (rotate (xyz 0 0 0))
-    )
-  )
   (module Resistors_THT:R_Axial_DIN0204_L3.6mm_D1.6mm_P5.08mm_Horizontal (layer F.Cu)
     (at 209.55 104.2162 180)
@@
       (net 4 "Net-(BT1-Pad2)"))
     (pad 3 thru_hole circle (at -5 -1.6 180) (size 1.5 1.5) (drill 0.9) (layers F.Cu F.Mask))
+  )
+  (module Transistors_OldSowjetAera:OldSowjetaera_Transistor_Type-II_SmallPads (layer F.Cu)
+    (at 219.46768 108.56214 270)
+    (fp_text reference Q1 (at 0 -7.1 270) (layer F.SilkS)
+      (effects (font (size 1 1) (thickness 0.15)))
+    )
+    (fp_text value BC547 (at 0.1 7.6 270) (layer F.Fab)
+      (effects (font (size 1 1) (thickness 0.15)))
+    )
+    (fp_circle (center -4.8 0) (end -4.8 0.4) (layer F.SilkS) (width 0.15))
+    (fp_circle (center 0 0) (end 4 0) (layer F.SilkS) (width 0.15))
+    (fp_circle (center 0 0) (end 5.6 0) (layer F.SilkS) (width 0.15))
+    (pad 2 thru_hole circle (at 0 -2 270) (size 1.6 1.6) (drill 0.8) (layers *.Cu *.Mask)
+      (net 2 "Net-(C1-Pad2)"))
+    (pad 1 thru_hole circle (at -2 0 270) (size 1.6 1.6) (drill 0.8) (layers *.Cu *.Mask)
+      (net 3 "Net-(C2-Pad1)"))
+    (pad 3 thru_hole circle (at 2 0 270) (size 1.6 1.6) (drill 0.8) (layers *.Cu *.Mask)
+      (net 6 "Net-(Q1-Pad3)"))
+    (model Transistors_OldSowjetAera.3dshapes/OldSowjetaera_Transistor_Type-II_SmallPads.wrl
+      (at (xyz 0 0 0))
+      (scale (xyz 0.3937 0.3937 0.3937))
+      (rotate (xyz 0 0 0))
+    )
   )
   (gr_text "Ivars & KO" (at 210.4136 119.0752) (layer F.SilkS)
@@
   (segment (start 204.47 100.33) (end 199.8358 100.33) (width 0.1) (layer F.Cu) (net 2))
   (segment (start 199.8358 100.33) (end 199.771 100.2652) (width 0.1) (layer F.Cu) (net 2))
+  (segment (start 219.47 100.33) (end 219.47 106.55982) (width 0.1) (layer F.Cu) (net 3))
+  (segment (start 219.47 106.55982) (end 219.46768 106.56214) (width 0.1) (layer F.Cu) (net 3))
   (segment (start 211.2772 104.2162) (end 213.6206 106.5596) (width 0.1) (layer F.Cu) (net 3))
   (segment (start 213.6206 106.5596) (end 219.4814 106.5596) (width 0.1) (layer F.Cu) (net 3))
